File: USB2serial.kicad_sch (KiCad schematic)
At the start: 7 parts, among them J2 Conn_02x03_Odd_Even, Q1 MMDT2222A, SW1 SW_Push, U5 CP2102N-Axx-xQFN28

Commit message: wip
Parts:
- removed Q1: MMDT2222A, Package_TO_SOT_SMD:SOT-363_SC-70-6, symbol Transistor_BJT:MMDT2222A
- added Q1, Q2: MMBT3904, Package_TO_SOT_SMD:SOT-23, symbol Transistor_BJT:MMBT3904
- J2: footprint (none) -> Connector_PinSocket_2.54mm:PinSocket_2x03_P2.54mm_Vertical
Connections:
- net CHIP_PU: now also Q1.3 (C)
- net DTR: now also Q2.2 (E)
- net IO0: now also Q2.3 (C)
- net RTS: now also Q1.2 (E)
- net at R8.1: now also Q2.1 (B)
- net at R7.1: now also Q1.1 (B)
Changed lines of the file:
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@@
     (pin "2")
+  )
+  (symbol (lib_id "Transistor_BJT:MMBT3904") (at 187.706 105.156 0) (mirror x) (unit 1)
+    (in_bom yes) (on_board yes) (fields_autoplaced)
+    (property "Reference" "Q2" (id 0) (at 193.04 103.8859 0)
+      (effects (font (size 1.27 1.27)) (justify left))
+    )
+    (property "Value" "MMBT3904" (id 1) (at 193.04 106.4259 0)
+      (effects (font (size 1.27 1.27)) (justify left))
+    )
+    (property "Footprint" "Package_TO_SOT_SMD:SOT-23" (id 2) (at 192.786 103.251 0)
+      (effects (font (size 1.27 1.27) italic) (justify left) hide)
+    )
+    (property "Datasheet" "https://datasheet.lcsc.com/lcsc/1811011934_Jiangsu-Changjing-Electronics-Technology-Co---Ltd--MMBT3904_C20526.pdf" (id 3) (at 187.706 105.156 0)
+      (effects (font (size 1.27 1.27)) (justify left) hide)
+    )
+    (pin "1")
+    (pin "2")
+    (pin "3")
   )
   (symbol (lib_id "Switch:SW_Push") (at 194.056 121.666 0) (unit 1)
@@
     (pin "2")
   )
+  (symbol (lib_id "Transistor_BJT:MMBT3904") (at 187.706 89.916 0) (unit 1)
+    (in_bom yes) (on_board yes) (fields_autoplaced)
+    (property "Reference" "Q1" (id 0) (at 193.04 88.6459 0)
+      (effects (font (size 1.27 1.27)) (justify left))
+    )
+    (property "Value" "MMBT3904" (id 1) (at 193.04 91.1859 0)
+      (effects (font (size 1.27 1.27)) (justify left))
+    )
+    (property "Footprint" "Package_TO_SOT_SMD:SOT-23" (id 2) (at 192.786 91.821 0)
+      (effects (font (size 1.27 1.27) italic) (justify left) hide)
+    )
+    (property "Datasheet" "https://datasheet.lcsc.com/lcsc/1811011934_Jiangsu-Changjing-Electronics-Technology-Co---Ltd--MMBT3904_C20526.pdf" (id 3) (at 187.706 89.916 0)
+      (effects (font (size 1.27 1.27)) (justify left) hide)
+    )
+    (pin "1")
+    (pin "2")
+    (pin "3")
+  )
   (symbol (lib_id "esp32_prog_board-rescue:+3.3V-power") (at 214.376 120.396 0) (unit 1)
     (in_bom yes) (on_board yes)
@@
     (pin "1")
   )
-  (symbol (lib_id "Transistor_BJT:MMDT2222A") (at 187.706 89.916 0) (unit 1)
-    (in_bom yes) (on_board yes)
-    (property "Reference" "Q1" (id 0) (at 192.532 88.7476 0)
-      (effects (font (size 1.27 1.27)) (justify left))
-    )
-    (property "Value" "MMDT2222A" (id 1) (at 192.532 91.059 0)
-      (effects (font (size 1.27 1.27)) (justify left))
-    )
-    (property "Footprint" "Package_TO_SOT_SMD:SOT-363_SC-70-6" (id 2) (at 192.786 87.376 0)
-      (effects (font (size 1.27 1.27)) hide)
-    )
-    (property "Datasheet" "http://www.diodes.com/_files/datasheets/ds30125.pdf" (id 3) (at 187.706 89.916 0)
-      (effects (font (size 1.27 1.27)) hide)
-    )
-    (pin "1")
-    (pin "2")
-    (pin "6")
-    (pin "3")
-    (pin "4")
-    (pin "5")
-  )
-  (symbol (lib_id "Transistor_BJT:MMDT2222A") (at 187.706 105.156 0) (mirror x) (unit 2)
-    (in_bom yes) (on_board yes)
-    (property "Reference" "Q1" (id 0) (at 192.532 103.9876 0)
-      (effects (font (size 1.27 1.27)) (justify left))
-    )
-    (property "Value" "MMDT2222A" (id 1) (at 192.532 106.299 0)
-      (effects (font (size 1.27 1.27)) (justify left))
-    )
-    (property "Footprint" "Package_TO_SOT_SMD:SOT-363_SC-70-6" (id 2) (at 192.786 107.696 0)
-      (effects (font (size 1.27 1.27)) hide)
-    )
-    (property "Datasheet" "http://www.diodes.com/_files/datasheets/ds30125.pdf" (id 3) (at 187.706 105.156 0)
-      (effects (font (size 1.27 1.27)) hide)
-    )
-    (pin "1")
-    (pin "2")
-    (pin "6")
-    (pin "3")
-    (pin "4")
-    (pin "5")
-  )
   (symbol (lib_id "power:GND") (at 121.158 150.114 0) (unit 1)
     (in_bom yes) (on_board yes)
@@
     (property "Reference" "J2" (id 0) (at 256.794 93.98 0))
     (property "Value" "Conn_02x03_Odd_Even" (id 1) (at 256.794 96.52 0))
-    (property "Footprint" "" (id 2) (at 255.524 103.378 0)
+    (property "Footprint" "Connector_PinSocket_2.54mm:PinSocket_2x03_P2.54mm_Vertical" (id 2) (at 255.524 103.378 0)
       (effects (font (size 1.27 1.27)) hide)
     )

Commit message: feature creep
Parts:
- added C11, C13: 2.2u, Capacitor_SMD:C_0805_2012Metric, symbol Device:C
- added C12, C14: 100n, Capacitor_SMD:C_0402_1005Metric, symbol Device:C
- R9: footprint Resistor_SMD:R_0402_1005Metric -> Resistor_SMD:R_0603_1608Metric
Connections:
- net +3V3: now also C13.1, C14.1
- net GND: now also C11.2, C12.2, C13.2, C14.2
- net +5V renamed VIN
- net VIN: now also C11.1, C12.1

Commit message: ready for JLCPCB
Parts:
- added 3V3: TestPoint, TestPoint:TestPoint_Pad_D1.0mm, symbol Connector:TestPoint
- added D3: LED_GREEN, LED_SMD:LED_0603_1608Metric, symbol Device:LED
- added R16: 22k, Resistor_SMD:R_0402_1005Metric, symbol Device:R
- added R17: 47k, Resistor_SMD:R_0402_1005Metric, symbol Device:R
- added R18: 4k7, Resistor_SMD:R_0402_1005Metric, symbol Device:R
- added R19: 220R, Resistor_SMD:R_0402_1005Metric, symbol Device:R
- J2: now left out of the parts list
Connections:
- net +3V3: now also 3V3.1, R18.1
- net GND: now also D3.1 (K), R17.2
- net VIN: now also R16.1; no longer U5.8 (VBUS)
- net at U5.11 (~{SUSPEND}): now also R19.1
- net at U5.9 (~{RST}): now also R18.2
- new net: D3.2 (A), R19.2
- new net: R16.2, R17.1, U5.8 (VBUS)
- no-connect marks 10 -> 15
