File: Boost.kicad_sch (KiCad schematic)
At the start: 16 parts, among them J3 Conn_01x02, U2 MC34063AD

Commit message: feature creep
Parts:
- removed C3: 330u/35V, Capacitor_THT:CP_Radial_D10.0mm_P5.00mm, symbol Device:C_Polarized
- removed C4: 100u/35V, Capacitor_THT:CP_Radial_D6.3mm_P2.50mm, symbol Device:C_Polarized
- added C10, C3, C4, C7, C8, C9: 22u/25V, Capacitor_SMD:C_1206_3216Metric, symbol Device:C
- added C6: 100n, Capacitor_SMD:C_0402_1005Metric, symbol Device:C
- added Q3: AO3401A, Package_TO_SOT_SMD:SOT-23, symbol Transistor_FET:AO3401A
- added R14: 100k, Resistor_SMD:R_0402_1005Metric, symbol Device:R
- added R15: 4k7, Resistor_SMD:R_0402_1005Metric, symbol Device:R
- C1, C5: value 10u/50V -> 22u/25V; footprint Capacitor_SMD:C_0805_2012Metric -> Capacitor_SMD:C_1206_3216Metric; LCSC C440198 -> C12891
- C2: value 680p -> 330p; LCSC C1630 -> C1664
- L1: value 68uH/1.2A -> 47uH/1.6A; footprint Local:NR8040T680M -> Local:PM3316680MRC; LCSC C223044 -> C1329349
- R11: footprint Resistor_SMD:R_0402_1005Metric -> Resistor_SMD:R_0805_2012Metric; LCSC C25765 -> C4328
- R3, R4, R5, R6: footprint Resistor_SMD:R_0402_1005Metric -> Resistor_SMD:R_0805_2012Metric; LCSC C25086 -> C25271
Connections:
- net +24V: now also C3.1, C4.1
- net GND: now also C10.2, C3.2, C4.2, C7.2, C8.2, C9.2, R15.2
- net VBUS: now also Q3.2 (S), R14.1; no longer C1.1, R3.2, R4.2, R5.2, R6.2, U2.6 (Vin)
- new net: C6.2, Q3.1 (G), R14.2, R15.1
- new net VIN: C1.1, C10.1, C6.1, C7.1, C8.1, C9.1, Q3.3 (D), R3.2, R4.2, R5.2, R6.2, U2.6 (Vin)
Other:
- note added: "Vout: 21V Vin: 4.5V Ct: 323pF Ipeak: 1A Rsc: 0.29Ohm Lmin: 31uH Co: 48uF"
- note added: "see AN920-D"
- note added: "see AN_146_USB_Hardware_Design_Guidelines_for_FTDI_ICs section 2.4.2"
- moved on the sheet: J3

Commit message: ready for JLCPCB
Parts:
- added VIN1: TestPoint, TestPoint:TestPoint_Pad_D1.0mm, symbol Connector:TestPoint
- J3: now left out of the parts list
- R15: LCSC (none) -> C25900
Connections:
- net VIN: now also VIN1.1
Changed lines of the file:
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@@
     (pin "2")
+  )
+  (symbol (lib_id "Connector:TestPoint") (at 92.202 90.678 0) (unit 1)
+    (in_bom yes) (on_board yes) (fields_autoplaced)
+    (property "Reference" "VIN1" (id 0) (at 94.488 86.1059 0)
+      (effects (font (size 1.27 1.27)) (justify left))
+    )
+    (property "Value" "TestPoint" (id 1) (at 94.488 88.6459 0)
+      (effects (font (size 1.27 1.27)) (justify left))
+    )
+    (property "Footprint" "TestPoint:TestPoint_Pad_D1.0mm" (id 2) (at 97.282 90.678 0)
+      (effects (font (size 1.27 1.27)) hide)
+    )
+    (property "Datasheet" "~" (id 3) (at 97.282 90.678 0)
+      (effects (font (size 1.27 1.27)) hide)
+    )
+    (pin "1")
   )
   (symbol (lib_id "Device:C") (at 225.298 102.616 0) (unit 1)
@@
   )
   (symbol (lib_id "Connector_Generic:Conn_01x02") (at 259.588 102.108 0) (unit 1)
-    (in_bom yes) (on_board yes) (fields_autoplaced)
+    (in_bom no) (on_board yes) (fields_autoplaced)
     (property "Reference" "J3" (id 0) (at 261.874 103.3779 0)
       (effects (font (size 1.27 1.27)) (justify left))
@@
       (effects (font (size 1.27 1.27)) hide)
     )
+    (property "LCSC" "C25900" (id 4) (at 34.29 110.49 0)
+      (effects (font (size 1.27 1.27)) hide)
+    )

Commit message: this was sent to jlcpcb
Parts:
- D1: footprint Diode_SMD:D_SMC -> Diode_SMD:D_SMA
Changed lines of the file:
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@@
     (property "Reference" "D1" (id 0) (at 187.2615 88.9 0))
     (property "Value" "D_Schottky" (id 1) (at 187.2615 91.44 0))
-    (property "Footprint" "Diode_SMD:D_SMC" (id 2) (at 186.944 95.758 0)
+    (property "Footprint" "Diode_SMD:D_SMA" (id 2) (at 186.944 95.758 0)
       (effects (font (size 1.27 1.27)) hide)
     )
