File: Esp32PWP.kicad_pcb (KiCad board)
At the start: 2 copper layers, 24 parts, among them Q1 MMDT2222A, U1 SRV05-4, U2 STUSB4500QTR, U3 STM32L151C8Tx, U4 STM32F030C8Tx, U5 CP2102N-Axx-xQFN28

Commit message: wip
Parts:
- removed D3: LED_BLUE, LED_SMD:LED_0603_1608Metric
- removed U3: STM32L151C8Tx, Package_QFP:LQFP-48_7x7mm_P0.5mm
- removed U4: STM32F030C8Tx, Package_QFP:LQFP-48_7x7mm_P0.5mm
- added C4: 100u/35V, Capacitor_THT:CP_Radial_D6.3mm_P2.50mm, F.Cu at (116.0, 50.0)
- added C5: 10u/50V, Capacitor_SMD:C_0805_2012Metric, F.Cu at (133.0, 42.2)
- added D1: D_Schottky, Diode_SMD:D_SMC, F.Cu at (144.5, 48.5)
- added F1: 2920L150DR, Fuse:Fuse_2920_7451Metric, F.Cu at (134.0, 68.0)
- added J1: HRO-TYPE-C-31-M-12, Local:HRO-TYPE-C-31-M-12, F.Cu at (111.9, 58.0)
- added J2: Conn_02x03_Odd_Even, Connector_PinSocket_2.54mm:PinSocket_2x03_P2.54mm_Vertical, F.Cu at (165.3, 58.5)
- added J3: Conn_01x02, Local:1985807, F.Cu at (163.4, 49.0)
- added L1: 68uH/1.2A, Local:NR8040T680M, F.Cu at (135.8, 48.5)
- added Q2: MMBT3904, Package_TO_SOT_SMD:SOT-23, F.Cu at (144.1, 60.0)
- added R10: 180R, Resistor_SMD:R_0603_1608Metric, F.Cu at (124.5, 50.8)
- added R11: 20k, Resistor_SMD:R_0402_1005Metric, F.Cu at (133.0, 40.5)
- added R12: 1.2k, Resistor_SMD:R_0402_1005Metric, F.Cu at (129.2, 41.5)
- added R13: 2.7k, Resistor_SMD:R_0402_1005Metric, F.Cu at (121.0, 66.2)
- added SW1: SW_Push, Local:TS-1187A-B-A-B, F.Cu at (155.0, 67.0)
- C1: value 1u/25V -> 10u/50V; footprint Capacitor_SMD:C_0402_1005Metric -> Capacitor_SMD:C_0805_2012Metric
- C2: value 1u/25V -> 680p; footprint Capacitor_SMD:C_0402_1005Metric -> Capacitor_SMD:C_0603_1608Metric
- C3: value 1u/25V -> 330u/35V; footprint Capacitor_SMD:C_0402_1005Metric -> Capacitor_THT:CP_Radial_D10.0mm_P5.00mm
- Q1: value MMDT2222A -> MMBT3904; footprint Package_TO_SOT_SMD:SOT-363_SC-70-6 -> Package_TO_SOT_SMD:SOT-23
- R1: value 10k -> 5.1k
- R2: value 100k -> 5.1k
- R3: value 470R -> 1R
- R4: value 1k -> 1R
- R5: value 100k -> 1R
- R6: value 200R -> 1R
- U2: value STUSB4500QTR -> MC34063AD; footprint Package_DFN_QFN:QFN-24-1EP_4x4mm_P0.5mm_EP2.7x2.7mm -> Package_SO:SOIC-8_3.9x4.9mm_P1.27mm
- moved C2 63.6 mm to (129.2, 43.2), turned to 180 degrees
- moved C3 60.6 mm to (153.2, 46.2), turned to -90 degrees
- moved H3 60.4 mm to (115.0, 42.0)
- moved R5 57.9 mm to (121.7, 49.0), turned to 180 degrees
- moved H4 56.3 mm to (166.0, 42.0)
- moved R3 55.4 mm to (121.8, 51.5), turned to 180 degrees
- moved C1 54.4 mm to (121.8, 45.2), turned to 90 degrees
- moved R4 53.1 mm to (121.8, 50.2), turned to 180 degrees
- moved U2 51.9 mm to (126.8, 47.0), turned to 180 degrees
- moved R6 50.1 mm to (121.8, 47.8), turned to 180 degrees
- moved H1 49.5 mm to (166.0, 69.0)
- moved R1 41.9 mm to (127.0, 65.0)
- moved R2 39.5 mm to (126.0, 56.0), turned to 180 degrees
- moved R7 39.2 mm to (146.8, 56.5)
- moved U5 38.6 mm to (134.0, 60.5), turned to 180 degrees
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Connections:
- C1 pad 1: Net-(C1-Pad1) -> VBUS
- C3 pad 1: Net-(C3-Pad1) -> +24V
- D2 pad 1: unconnected-(D2-Pad1) -> GND
- D2 pad 2: unconnected-(D2-Pad2) -> Net-(D2-Pad2)
- Q1 pad 1: /USB2serial/RTS -> Net-(R7-Pad1)
- Q1 pad 2: Net-(Q1-Pad2) -> /USB2serial/RTS
- Q1 pad 3: /USB2serial/IO0 -> /USB2serial/CHIP_PU
- R1 pad 1: Net-(R1-Pad1) -> /CC2
- R2 pad 1: Net-(R2-Pad1) -> /CC1
- R3 pad 1: VBUS -> Net-(L1-Pad1)
- R3 pad 2: Net-(C1-Pad1) -> VBUS
- R4 pad 1: Net-(C1-Pad1) -> Net-(L1-Pad1)
- R4 pad 2: Net-(R4-Pad2) -> VBUS
- R5 pad 1: Net-(R5-Pad1) -> Net-(L1-Pad1)
- R5 pad 2: GND -> VBUS
- R6 pad 1: VBUS -> Net-(L1-Pad1)
- R6 pad 2: Net-(R6-Pad2) -> VBUS
- R7 pad 1: Net-(Q1-Pad2) -> Net-(R7-Pad1)
- R8 pad 1: Net-(Q1-Pad5) -> Net-(R8-Pad1)
- U1 pad 5: +5V -> VBUS
- U2 pad 1: /CC1 -> Net-(D1-Pad2)
- U2 pad 2: /CC1 -> GND
- U2 pad 3: unconnected-(U2-Pad3) -> Net-(C2-Pad1)
- U2 pad 4: /CC2 -> GND
- U2 pad 5: /CC2 -> Net-(R11-Pad2)
- U2 pad 6: Net-(R1-Pad1) -> VBUS
- U2 pad 7: GND -> Net-(L1-Pad1)
- U2 pad 8: GND -> Net-(R10-Pad2)
Other:
- board outline added: 57 x 33 mm

Commit message: wip
Parts:
- added TP1: TestPoint, TestPoint:TestPoint_Pad_D2.0mm, F.Cu at (143.0, 70.0)
- added TP2: TestPoint, TestPoint:TestPoint_Pad_D2.0mm, F.Cu at (147.1, 70.0)
Changed lines of the file:
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@@
   (net 8 "unconnected-(J1-PadB8)")
   (net 9 "/USB2serial/RTS")
-  (net 10 "Net-(R7-Pad1)")
+  (net 10 "Net-(F1-Pad2)")
   (net 11 "/USB2serial/IO0")
   (net 12 "/USB2serial/DTR")
-  (net 13 "Net-(R8-Pad1)")
+  (net 13 "Net-(Q1-Pad1)")
   (net 14 "/USB2serial/CHIP_PU")
   (net 15 "Net-(D1-Pad2)")
@@
   (net 44 "/USB2serial/TX")
   (net 45 "unconnected-(U5-Pad27)")
-  (net 46 "Net-(J1-PadA4)")
+  (net 46 "Net-(Q2-Pad1)")
   (footprint "Resistor_SMD:R_0402_1005Metric" (layer "F.Cu")
     (at 133 40.5 180)
@@
     (fp_line (start -0.65 1.45) (end -0.65 -1.125) (layer "F.Fab") (width 0.1))
     (pad "1" smd roundrect (at -0.9375 -0.95) (size 1.475 0.6) (layers "F.Cu" "F.Paste" "F.Mask") (roundrect_rratio 0.25)
-      (net 13 "Net-(R8-Pad1)") (pinfunction "B") (pintype "input"))
+      (net 46 "Net-(Q2-Pad1)") (pinfunction "B") (pintype "input"))
     (pad "2" smd roundrect (at -0.9375 0.95) (size 1.475 0.6) (layers "F.Cu" "F.Paste" "F.Mask") (roundrect_rratio 0.25)
       (net 12 "/USB2serial/DTR") (pinfunction "E") (pintype "passive"))
@@
       (rotate (xyz 0 0 0))
     )
+  )
+  (footprint "TestPoint:TestPoint_Pad_D2.0mm" (layer "F.Cu")
+    (at 143 70)
+    (descr "SMD pad as test Point, diameter 2.0mm")
+    (tags "test point SMD pad")
+    (property "Sheetfile" "Esp32PWP.kicad_sch")
+    (property "Sheetname" "")
+    (attr exclude_from_pos_files)
+    (fp_text reference "TP1" (at 0 -1.998) (layer "F.SilkS")
+      (effects (font (size 1 1) (thickness 0.15)))
+    )
+    (fp_text value "TestPoint" (at 0 2.05) (layer "F.Fab")
+      (effects (font (size 1 1) (thickness 0.15)))
+    )
+    (fp_text user "${REFERENCE}" (at 0 -2) (layer "F.Fab")
+      (effects (font (size 1 1) (thickness 0.15)))
+    )
+    (fp_circle (center 0 0) (end 0 1.2) (layer "F.SilkS") (width 0.12) (fill none))
+    (fp_circle (center 0 0) (end 1.5 0) (layer "F.CrtYd") (width 0.05) (fill none))
+    (pad "1" smd circle (at 0 0) (size 2 2) (layers "F.Cu" "F.Mask")
+      (net 25 "/CC2") (pinfunction "1") (pintype "passive"))
   )
   (footprint "Package_TO_SOT_SMD:SOT-23-6" (layer "F.Cu")
@@
     (fp_line (start 0.525 0.27) (end -0.525 0.27) (layer "F.Fab") (width 0.1))
     (pad "1" smd roundrect (at -0.51 0) (size 0.54 0.64) (layers "F.Cu" "F.Paste" "F.Mask") (roundrect_rratio 0.25)
-      (net 13 "Net-(R8-Pad1)") (pintype "passive"))
+      (net 46 "Net-(Q2-Pad1)") (pintype "passive"))
     (pad "2" smd roundrect (at 0.51 0) (size 0.54 0.64) (layers "F.Cu" "F.Paste" "F.Mask") (roundrect_rratio 0.25)
       (net 9 "/USB2serial/RTS") (pintype "passive"))
@@
     (fp_line (start -0.325 -1.45) (end 0.65 -1.45) (layer "F.Fab") (width 0.1))
     (pad "1" smd roundrect (at -0.9375 -0.95) (size 1.475 0.6) (layers "F.Cu" "F.Paste" "F.Mask") (roundrect_rratio 0.25)
-      (net 10 "Net-(R7-Pad1)") (pinfunction "B") (pintype "input"))
+      (net 13 "Net-(Q1-Pad1)") (pinfunction "B") (pintype "input"))
     (pad "2" smd roundrect (at -0.9375 0.95) (size 1.475 0.6) (layers "F.Cu" "F.Paste" "F.Mask") (roundrect_rratio 0.25)
       (net 9 "/USB2serial/RTS") (pinfunction "E") (pintype "passive"))
@@
       (net 16 "VBUS") (pintype "passive"))
     (pad "2" smd roundrect (at 3.3875 0 180) (size 1.925 5.45) (layers "F.Cu" "F.Paste" "F.Mask") (roundrect_rratio 0.12987)
-      (net 46 "Net-(J1-PadA4)") (pintype "passive"))
+      (net 10 "Net-(F1-Pad2)") (pintype "passive"))
     (model "${KICAD6_3DMODEL_DIR}/Fuse.3dshapes/Fuse_2920_7451Metric.wrl"
       (offset (xyz 0 0 0))
@@
       (rotate (xyz 0 0 0))
     )
+  )
+  (footprint "TestPoint:TestPoint_Pad_D2.0mm" (layer "F.Cu")
+    (at 147.05 70)
+    (descr "SMD pad as test Point, diameter 2.0mm")
+    (tags "test point SMD pad")
+    (property "Sheetfile" "Esp32PWP.kicad_sch")
+    (property "Sheetname" "")
+    (attr exclude_from_pos_files)
+    (fp_text reference "TP2" (at 0 -1.998) (layer "F.SilkS")
+      (effects (font (size 1 1) (thickness 0.15)))
+    )
+    (fp_text value "TestPoint" (at 0 2.05) (layer "F.Fab")
+      (effects (font (size 1 1) (thickness 0.15)))
+    )
+    (fp_text user "${REFERENCE}" (at 0 -2) (layer "F.Fab")
+      (effects (font (size 1 1) (thickness 0.15)))
+    )
+    (fp_circle (center 0 0) (end 0 1.2) (layer "F.SilkS") (width 0.12) (fill none))
+    (fp_circle (center 0 0) (end 1.5 0) (layer "F.CrtYd") (width 0.05) (fill none))
+    (pad "1" smd circle (at 0 0) (size 2 2) (layers "F.Cu" "F.Mask")
+      (net 24 "/CC1") (pinfunction "1") (pintype "passive"))
   )
   (footprint "Resistor_SMD:R_0402_1005Metric" (layer "F.Cu")
@@
       (net 2 "GND") (pinfunction "GND") (pintype "passive"))
     (pad "A4" smd rect (at -2.45 -7.695 270) (size 0.6 1.45) (layers "F.Cu" "F.Paste" "F.Mask")
-      (net 46 "Net-(J1-PadA4)") (pinfunction "VBUS") (pintype "passive"))
+      (net 10 "Net-(F1-Pad2)") (pinfunction "VBUS") (pintype "passive"))
     (pad "A5" smd rect (at -1.25 -7.695 270) (size 0.3 1.45) (layers "F.Cu" "F.Paste" "F.Mask")
       (net 24 "/CC1") (pinfunction "CC1") (pintype "bidirectional"))
@@
       (net 8 "unconnected-(J1-PadB8)") (pinfunction "SBU2") (pintype "bidirectional+no_connect"))
     (pad "B9" smd rect (at 2.45 -7.695 270) (size 0.6 1.45) (layers "F.Cu" "F.Paste" "F.Mask")
-      (net 46 "Net-(J1-PadA4)") (pinfunction "VBUS") (pintype "passive"))
+      (net 10 "Net-(F1-Pad2)") (pinfunction "VBUS") (pintype "passive"))
     (pad "S1" thru_hole oval (at -4.32 -2.6 270) (size 1 1.6) (drill oval 0.6 1.2) (layers *.Cu "B.Mask")
       (net 2 "GND") (pinfunction "SHIELD") (pintype "passive"))
@@
     (fp_line (start 0.525 -0.27) (end 0.525 0.27) (layer "F.Fab") (width 0.1))
     (pad "1" smd roundrect (at -0.51 0) (size 0.54 0.64) (layers "F.Cu" "F.Paste" "F.Mask") (roundrect_rratio 0.25)
-      (net 10 "Net-(R7-Pad1)") (pintype "passive"))
+      (net 13 "Net-(Q1-Pad1)") (pintype "passive"))
     (pad "2" smd roundrect (at 0.51 0) (size 0.54 0.64) (layers "F.Cu" "F.Paste" "F.Mask") (roundrect_rratio 0.25)
       (net 12 "/USB2serial/DTR") (pintype "passive"))

Commit message: feature creep
Parts:
- added C10: 22u/25V, Capacitor_SMD:C_1206_3216Metric, F.Cu at (129.9, 42.0)
- added C11: 2.2u, Capacitor_SMD:C_0805_2012Metric, F.Cu at (139.9, 61.5)
- added C12: 100n, Capacitor_SMD:C_0402_1005Metric, F.Cu at (141.7, 61.7)
- added C13: 2.2u, Capacitor_SMD:C_0805_2012Metric, F.Cu at (158.1, 57.2)
- added C14: 100n, Capacitor_SMD:C_0402_1005Metric, F.Cu at (159.8, 57.7)
- added C6: 100n, Capacitor_SMD:C_0402_1005Metric, F.Cu at (123.3, 48.4)
- added C7: 22u/25V, Capacitor_SMD:C_1206_3216Metric, F.Cu at (132.4, 42.0)
- added C8: 22u/25V, Capacitor_SMD:C_1206_3216Metric, F.Cu at (127.4, 42.0)
- added C9: 22u/25V, Capacitor_SMD:C_1206_3216Metric, F.Cu at (124.9, 42.0)
- added J4: USB_A, Local:UE27AE54100, F.Cu at (134.0, 69.0)
- added J5: USB_A, Local:UE27AE54100, F.Cu at (134.0, 79.0)
- added Q3: AO3401A, Package_TO_SOT_SMD:SOT-23, F.Cu at (126.5, 48.1)
- added R14: 100k, Resistor_SMD:R_0402_1005Metric, F.Cu at (123.3, 49.6)
- added R15: 4k7, Resistor_SMD:R_0402_1005Metric, F.Cu at (123.3, 47.1)
- added TP3: TestPoint, TestPoint:TestPoint_Pad_D2.0mm, F.Cu at (117.5, 48.1)
- added U3: USB2514B_Bi, Package_DFN_QFN:QFN-36-1EP_6x6mm_P0.5mm_EP3.7x3.7mm, F.Cu at (152.7, 75.6)
- C1, C5: value 10u/50V -> 22u/25V; footprint Capacitor_SMD:C_0805_2012Metric -> Capacitor_SMD:C_1206_3216Metric
- C2: value 680p -> 330p
- C3: value 330u/35V -> 22u/25V; footprint Capacitor_THT:CP_Radial_D10.0mm_P5.00mm -> Capacitor_SMD:C_1206_3216Metric
- C4: value 100u/35V -> 22u/25V; footprint Capacitor_THT:CP_Radial_D6.3mm_P2.50mm -> Capacitor_SMD:C_1206_3216Metric
- L1: value 68uH/1.2A -> 47uH/1.6A; footprint Local:NR8040T680M -> Local:PM3316680MRC
- R11, R3, R4, R5, R6: footprint Resistor_SMD:R_0402_1005Metric -> Resistor_SMD:R_0805_2012Metric
- R9: footprint Resistor_SMD:R_0402_1005Metric -> Resistor_SMD:R_0603_1608Metric
- TP1, TP2: footprint TestPoint:TestPoint_Pad_D2.0mm -> TestPoint:TestPoint_Pad_D1.0mm
- moved C4 39.2 mm to (155.2, 48.2), turned to 0 degrees
- moved D2 36.4 mm to (154.8, 56.2), turned to 180 degrees
- moved TP2 25.3 mm to (123.5, 60.9)
- moved C5 23.8 mm to (155.2, 51.0), turned to 0 degrees
- moved TP1 21.9 mm to (125.2, 57.2)
- moved R13 17.6 mm to (135.8, 56.8), turned to 90 degrees
- moved C2 17.4 mm to (146.7, 42.8), turned to 90 degrees
- moved U2 15.4 mm to (141.9, 44.2)
- moved C1 13.6 mm to (134.9, 42.0)
- moved U5 12.1 mm to (145.8, 63.2), turned to -90 degrees
- moved R10 11.8 mm to (135.7, 47.0), turned to -90 degrees
- moved R6 11.4 mm to (132.9, 45.5)
- moved R5 11.3 mm to (132.9, 47.5)
- moved R4 11.2 mm to (132.9, 49.5)
- moved R3 11.2 mm to (132.9, 51.5)
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Connections:
- C1 pad 1: VBUS -> VIN
- C4 pad 1: VBUS -> +24V
- R13 pad 1: VBUS -> VIN
- R3 pad 2: VBUS -> VIN
- R4 pad 2: VBUS -> VIN
- R5 pad 2: VBUS -> VIN
- R6 pad 2: VBUS -> VIN
- U2 pad 6: VBUS -> VIN
- U5 pad 7: +5V -> VIN
- U5 pad 8: +5V -> VIN
Routing:
- net +24V: track 0.00 -> 34.5 mm
- net USB_D-: track 0.00 -> 31.2 mm, vias 0 -> 2
- net USB_D+: track 0.00 -> 31.2 mm
- net Net-(F1-Pad2): track 0.00 -> 29.2 mm
- net GND: track 0.00 -> 29.2 mm, vias 0 -> 2
- net /USB2serial/TX: track 0.00 -> 25.9 mm, vias 0 -> 1
- net +3V3: track 0.00 -> 22.7 mm, vias 0 -> 2
- net /USB2serial/IO0: track 0.00 -> 20.4 mm
- net /USB2serial/RX: track 0.00 -> 19.0 mm, vias 0 -> 1
- net Net-(D2-Pad2): track 0.00 -> 18.2 mm
- net /USB2serial/RTS: track 0.00 -> 15.7 mm, vias 0 -> 2
- net VBUS: track 0.00 -> 14.7 mm
- net VIN: track 0.00 -> 13.0 mm
- net /CC1: track 0.00 -> 13.0 mm
- net /USB2serial/DTR: track 0.00 -> 11.3 mm
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- added copper zone on F.Cu, net +24V
- added copper zone on B.Cu, net GND
- added copper zone on F.Cu, net GND
- added copper zone on F.Cu, net Net-(D1-Pad2)
- added copper zone on F.Cu, net Net-(L1-Pad1)
- added copper zone on F.Cu, net VIN
Other:
- board size 57 x 33 mm -> 54 x 44 mm
- board text added: "+21V"
- board text added: "3.3V EN GND RX IO0 TX"

Commit message: ready for JLCPCB
Parts:
- removed J4, J5: USB_A, Local:UE27AE54100
- removed U3: USB2514B_Bi, Package_DFN_QFN:QFN-36-1EP_6x6mm_P0.5mm_EP3.7x3.7mm
- added 3V3: TestPoint, TestPoint:TestPoint_Pad_D1.0mm, F.Cu at (138.8, 67.0)
- added D3: LED_GREEN, LED_SMD:LED_0603_1608Metric, F.Cu at (146.5, 68.0)
- added R16: 22k, Resistor_SMD:R_0402_1005Metric, F.Cu at (137.5, 62.0)
- added R17: 47k, Resistor_SMD:R_0402_1005Metric, F.Cu at (137.5, 64.2)
- added R18: 4k7, Resistor_SMD:R_0402_1005Metric, F.Cu at (141.5, 63.8)
- added R19: 220R, Resistor_SMD:R_0402_1005Metric, F.Cu at (143.5, 68.0)
- added VIN1: TestPoint, TestPoint:TestPoint_Pad_D1.0mm, F.Cu at (128.6, 45.4)
- R13: footprint Resistor_SMD:R_0402_1005Metric -> Resistor_SMD:R_0603_1608Metric
- moved C12 1.22 mm to (141.5, 60.5)
- moved C13 0.50 mm to (158.1, 56.8)
- moved C11 0.31 mm to (139.7, 61.2)
- moved R13 0.22 mm to (135.7, 57.0)
- moved L1 0.21 mm to (144.2, 53.0)
- moved C14 0.10 mm to (159.8, 57.6)
- renumbered TP2 to CC1, TP1 to CC2, TP3 to GND1
Connections:
- U5 pad 11: unconnected-(U5-Pad11) -> Net-(R19-Pad1)
- U5 pad 8: VIN -> Net-(R16-Pad2)
- U5 pad 9: unconnected-(U5-Pad9) -> Net-(R18-Pad2)
Routing:
- net GND: track 29.2 -> 54.7 mm, vias 2 -> 30
- net VIN: track 13.0 -> 25.9 mm, vias 0 -> 2
- net Net-(R16-Pad2): track 0.00 -> 11.5 mm
- net +3V3: track 22.7 -> 33.7 mm, vias 2 -> 3
- net +24V: track 34.5 -> 45.1 mm
- net Net-(R19-Pad1): track 0.00 -> 6.23 mm
- net /USB2serial/TX: track 25.9 -> 22.0 mm, vias 1 -> 2
- net Net-(R18-Pad2): track 0.00 -> 2.35 mm
- net Net-(D3-Pad2): track 0.00 -> 1.70 mm
- net /USB2serial/IO0: track 20.4 -> 21.8 mm
- net USB_D-: track 31.2 -> 30.4 mm
- net VBUS: track 14.7 -> 13.9 mm
Other:
- board size 54 x 44 mm -> 54 x 33 mm

Commit message: this was sent to jlcpcb
Parts:
- D1: footprint Diode_SMD:D_SMC -> Diode_SMD:D_SMA
- moved D1 0.76 mm to (151.9, 43.2)
Routing:
- net +24V: track 45.1 -> 46.3 mm
Changed lines of the file:
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@@
     )
   )
-  (footprint "Diode_SMD:D_SMC" (layer "F.Cu")
-    (at 152.6625 43.25 180)
-    (descr "Diode SMC (DO-214AB)")
-    (tags "Diode SMC (DO-214AB)")
+  (footprint "Diode_SMD:D_SMA" (layer "F.Cu")
+    (at 151.9 43.2 180)
+    (descr "Diode SMA (DO-214AC)")
+    (tags "Diode SMA (DO-214AC)")
     (property "LCSC" "C22452")
     (property "Sheetfile" "Boost.kicad_sch")
     (property "Sheetname" "Boost")
     (attr smd)
-    (fp_text reference "D1" (at -6.0875 2.75 180) (layer "F.SilkS")
-      (effects (font (size 1 1) (thickness 0.15)))
-    )
-    (fp_text value "D_Schottky" (at 0 4.2) (layer "F.Fab")
-      (effects (font (size 1 1) (thickness 0.15)))
-    )
-    (fp_text user "${REFERENCE}" (at 0 -1.9) (layer "F.Fab")
-      (effects (font (size 1 1) (thickness 0.15)))
-    )
-    (fp_line (start -4.8 3.25) (end 3.6 3.25) (layer "F.SilkS") (width 0.12))
-    (fp_line (start -4.8 3.25) (end -4.8 -3.25) (layer "F.SilkS") (width 0.12))
-    (fp_line (start -4.8 -3.25) (end 3.6 -3.25) (layer "F.SilkS") (width 0.12))
-    (fp_line (start -4.9 3.35) (end -4.9 -3.35) (layer "F.CrtYd") (width 0.05))
-    (fp_line (start 4.9 3.35) (end -4.9 3.35) (layer "F.CrtYd") (width 0.05))
-    (fp_line (start -4.9 -3.35) (end 4.9 -3.35) (layer "F.CrtYd") (width 0.05))
-    (fp_line (start 4.9 -3.35) (end 4.9 3.35) (layer "F.CrtYd") (width 0.05))
+    (fp_text reference "D1" (at 0 -2.5 180) (layer "F.SilkS")
+      (effects (font (size 1 1) (thickness 0.15)))
+    )
+    (fp_text value "D_Schottky" (at 0 2.6 180) (layer "F.Fab")
+      (effects (font (size 1 1) (thickness 0.15)))
+    )
+    (fp_text user "${REFERENCE}" (at 0 -2.5 180) (layer "F.Fab")
+      (effects (font (size 1 1) (thickness 0.15)))
+    )
+    (fp_line (start -3.4 -1.65) (end 2 -1.65) (layer "F.SilkS") (width 0.12))
+    (fp_line (start -3.4 1.65) (end 2 1.65) (layer "F.SilkS") (width 0.12))
+    (fp_line (start -3.4 -1.65) (end -3.4 1.65) (layer "F.SilkS") (width 0.12))
+    (fp_line (start -3.5 1.75) (end -3.5 -1.75) (layer "F.CrtYd") (width 0.05))
+    (fp_line (start 3.5 -1.75) (end 3.5 1.75) (layer "F.CrtYd") (width 0.05))
+    (fp_line (start 3.5 1.75) (end -3.5 1.75) (layer "F.CrtYd") (width 0.05))
+    (fp_line (start -3.5 -1.75) (end 3.5 -1.75) (layer "F.CrtYd") (width 0.05))
+    (fp_line (start 2.3 1.5) (end -2.3 1.5) (layer "F.Fab") (width 0.1))
+    (fp_line (start -0.64944 0.00102) (end -1.55114 0.00102) (layer "F.Fab") (width 0.1))
     (fp_line (start -0.64944 0.00102) (end 0.50118 -0.79908) (layer "F.Fab") (width 0.1))
+    (fp_line (start 2.3 -1.5) (end 2.3 1.5) (layer "F.Fab") (width 0.1))
+    (fp_line (start 2.3 -1.5) (end -2.3 -1.5) (layer "F.Fab") (width 0.1))
     (fp_line (start -0.64944 -0.79908) (end -0.64944 0.80112) (layer "F.Fab") (width 0.1))
-    (fp_line (start 3.55 -3.1) (end -3.55 -3.1) (layer "F.Fab") (width 0.1))
+    (fp_line (start 0.50118 0.75032) (end 0.50118 -0.79908) (layer "F.Fab") (width 0.1))
     (fp_line (start 0.50118 0.00102) (end 1.4994 0.00102) (layer "F.Fab") (width 0.1))
-    (fp_line (start 3.55 3.1) (end -3.55 3.1) (layer "F.Fab") (width 0.1))
-    (fp_line (start -0.64944 0.00102) (end -1.55114 0.00102) (layer "F.Fab") (width 0.1))
-    (fp_line (start -3.55 3.1) (end -3.55 -3.1) (layer "F.Fab") (width 0.1))
-    (fp_line (start 3.55 -3.1) (end 3.55 3.1) (layer "F.Fab") (width 0.1))
-    (fp_line (start 0.50118 0.75032) (end 0.50118 -0.79908) (layer "F.Fab") (width 0.1))
+    (fp_line (start -2.3 1.5) (end -2.3 -1.5) (layer "F.Fab") (width 0.1))
     (fp_line (start -0.64944 0.00102) (end 0.50118 0.75032) (layer "F.Fab") (width 0.1))
-    (pad "1" smd rect (at -3.4 0 270) (size 3.3 2.5) (layers "F.Cu" "F.Paste" "F.Mask")
+    (pad "1" smd rect (at -2 0 180) (size 2.5 1.8) (layers "F.Cu" "F.Paste" "F.Mask")
       (net 5 "+24V") (pinfunction "K") (pintype "passive"))
-    (pad "2" smd rect (at 3.4 0 270) (size 3.3 2.5) (layers "F.Cu" "F.Paste" "F.Mask")
+    (pad "2" smd rect (at 2 0 180) (size 2.5 1.8) (layers "F.Cu" "F.Paste" "F.Mask")
       (net 15 "Net-(D1-Pad2)") (pinfunction "A") (pintype "passive"))
-    (model "${KICAD6_3DMODEL_DIR}/Diode_SMD.3dshapes/D_SMC.wrl"
+    (model "${KICAD6_3DMODEL_DIR}/Diode_SMD.3dshapes/D_SMA.wrl"
       (offset (xyz 0 0 0))
       (scale (xyz 1 1 1))
@@
   (segment (start 139.4125 46.18) (end 139.4125 46.75) (width 0.25) (layer "F.Cu") (net 4))
   (segment (start 139.4375 46.155) (end 139.4125 46.18) (width 0.25) (layer "F.Cu") (net 4))
-  (segment (start 164.2 49.125) (end 164.125 49.125) (width 2) (layer "F.Cu") (net 5))
   (segment (start 132.9875 52.188173) (end 136.299327 55.5) (width 0.25) (layer "F.Cu") (net 5))
   (segment (start 151.9375 55.5) (end 153.6875 53.75) (width 0.25) (layer "F.Cu") (net 5))
-  (segment (start 164.125 49.125) (end 158.25 43.25) (width 2) (layer "F.Cu") (net 5))
   (segment (start 132.9875 44.811827) (end 132.9875 52.188173) (width 0.25) (layer "F.Cu") (net 5))
   (segment (start 137.1625 44.4125) (end 133.386827 44.4125) (width 0.25) (layer "F.Cu") (net 5))
-  (segment (start 158.25 43.25) (end 156.0625 43.25) (width 2) (layer "F.Cu") (net 5))
+  (segment (start 164.2 49.125) (end 164.125 49.125) (width 2) (layer "F.Cu") (net 5))
+  (segment (start 158.25 43.25) (end 154.8 43.25) (width 2) (layer "F.Cu") (net 5))
+  (segment (start 164.125 49.125) (end 158.25 43.25) (width 2) (layer "F.Cu") (net 5))
   (segment (start 133.386827 44.4125) (end 132.9875 44.811827) (width 0.25) (layer "F.Cu") (net 5))
   (segment (start 136.299327 55.5) (end 151.9375 55.5) (width 0.25) (layer "F.Cu") (net 5))
