File: Esp32PWP.kicad_sch (KiCad schematic)
At the start: 21 parts, among them J1 105450-0101, U1 SRV05-4, U2 STUSB4500QTR, U3 STM32L151C8Tx, U4 STM32F030C8Tx

Commit message: smth
Parts:
- added U?: USB2514B_Bi, Package_DFN_QFN:QFN-36-1EP_6x6mm_P0.5mm_EP3.7x3.7mm, symbol Interface_USB:USB2514B_Bi
Changed lines of the file:
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@@
     (pin "1")
+  )
+  (symbol (lib_id "Interface_USB:USB2514B_Bi") (at -93.726 95.504 0) (unit 1)
+    (in_bom yes) (on_board yes) (fields_autoplaced)
+    (property "Reference" "U?" (id 0) (at -91.7066 133.35 0)
+      (effects (font (size 1.27 1.27)) (justify left))
+    )
+    (property "Value" "USB2514B_Bi" (id 1) (at -91.7066 135.89 0)
+      (effects (font (size 1.27 1.27)) (justify left))
+    )
+    (property "Footprint" "Package_DFN_QFN:QFN-36-1EP_6x6mm_P0.5mm_EP3.7x3.7mm" (id 2) (at -60.706 133.604 0)
+      (effects (font (size 1.27 1.27)) hide)
+    )
+    (property "Datasheet" "http://ww1.microchip.com/downloads/en/DeviceDoc/00001692C.pdf" (id 3) (at -53.086 136.144 0)
+      (effects (font (size 1.27 1.27)) hide)
+    )
+    (pin "1")
+    (pin "10")
+    (pin "11")
+    (pin "12")
+    (pin "13")
+    (pin "14")
+    (pin "15")
+    (pin "16")
+    (pin "17")
+    (pin "18")
+    (pin "19")
+    (pin "2")
+    (pin "20")
+    (pin "21")
+    (pin "22")
+    (pin "23")
+    (pin "24")
+    (pin "25")
+    (pin "26")
+    (pin "27")
+    (pin "28")
+    (pin "29")
+    (pin "3")
+    (pin "30")
+    (pin "31")
+    (pin "32")
+    (pin "33")
+    (pin "34")
+    (pin "35")
+    (pin "36")
+    (pin "37")
+    (pin "4")
+    (pin "5")
+    (pin "6")
+    (pin "7")
+    (pin "8")
+    (pin "9")
   )
   (symbol (lib_id "power:GND") (at 165.354 77.724 0) (mirror y) (unit 1)
@@
       (reference "U5") (unit 1) (value "CP2102N-Axx-xQFN28") (footprint "Package_DFN_QFN:QFN-28-1EP_5x5mm_P0.5mm_EP3.35x3.35mm")
     )
-  )
+    (path "/08e0979f-3817-48ba-a4c0-a02126e6e841"
+      (reference "U?") (unit 1) (value "USB2514B_Bi") (footprint "Package_DFN_QFN:QFN-36-1EP_6x6mm_P0.5mm_EP3.7x3.7mm")
+    )
+  )

Commit message: wip
Parts:
- removed C1, C2, C3: 1u/25V, Capacitor_SMD:C_0402_1005Metric, symbol Device:C
- removed D1: D_Zener, symbol Device:D_Zener
- removed D3: LED_BLUE, LED_SMD:LED_0603_1608Metric, symbol Device:LED
- removed J1: 105450-0101, Molex:105450-0101, symbol esp32_prog_board-rescue:USB_C_Receptacle_USB2.0-Connector
- removed R3: 470R, Resistor_SMD:R_0402_1005Metric, symbol Device:R
- removed R4: 1k, Resistor_SMD:R_0402_1005Metric, symbol Device:R
- removed R5: 100k, Resistor_SMD:R_0402_1005Metric, symbol Device:R
- removed R6: 200R, Resistor_SMD:R_0402_1005Metric, symbol Device:R
- removed U2: STUSB4500QTR, Package_DFN_QFN:QFN-24-1EP_4x4mm_P0.5mm_EP2.7x2.7mm, symbol Interface_USB:STUSB4500QTR
- removed U3: STM32L151C8Tx, Package_QFP:LQFP-48_7x7mm_P0.5mm, symbol MCU_ST_STM32L1:STM32L151C8Tx
- removed U4: STM32F030C8Tx, Package_QFP:LQFP-48_7x7mm_P0.5mm, symbol MCU_ST_STM32F0:STM32F030C8Tx
- removed U?: USB2514B_Bi, Package_DFN_QFN:QFN-36-1EP_6x6mm_P0.5mm_EP3.7x3.7mm, symbol Interface_USB:USB2514B_Bi
- added F1: 2920L150DR, Fuse:Fuse_2920_7451Metric, symbol Device:Polyfuse
- added J1: HRO-TYPE-C-31-M-12, Local:HRO-TYPE-C-31-M-12, symbol Connector:USB_C_Receptacle_USB2.0
- added R13: 2.7k, Resistor_SMD:R_0402_1005Metric, symbol Device:R
- R1: value 10k -> 5.1k
- R2: value 100k -> 5.1k
Connections:
- net +5V is gone; now on net VBUS: U1.5 (VP)
- net CC1: now also R2.1, J1.A5 (CC1)
- net CC2: now also R1.1, J1.B5 (CC2)
- net GND: now also D2.1 (K), J1.A1 (GND), J1.A12 (GND), J1.B1 (GND), J1.B12 (GND), J1.S1 (SHIELD)
- net USB_D+: now also J1.A6 (D+), J1.B6 (D+)
- net USB_D-: now also J1.A7 (D-), J1.B7 (D-)
- net VBUS: now also F1.1, R13.1
- net at D2.2 (A): now also R13.2
- new net: F1.2, J1.A4 (VBUS), J1.A9 (VBUS), J1.B4 (VBUS), J1.B9 (VBUS)
- no-connect marks 9 -> 2
Other:
- added sheet Boost (Boost.kicad_sch)
- note added: "A Type-C host with 3A capability will have 10 k pull-up to 5 V, a 1.5 A capability will be advertised with 22k pull-up, and the standard port capability (500 mA) will have 56 k pull-up."
- note added: "https://github.com/jenschr/USB-C-Connectors https://dubiouscreations.com/2021/04/06/designing-with-usb-c-lessons-learned/ https://flashgamer.com/blog/comments/implementing-usb-type-c-and-usb-3-1"
- note removed: "25V enough?"
- note removed: "RECHECK THIS"
- moved on the sheet: U1

Commit message: wip
Parts:
- added TP1, TP2, TP?: TestPoint, TestPoint:TestPoint_Pad_D2.0mm, symbol Connector:TestPoint
Connections:
- net CC1: now also TP2.1
- net CC2: now also TP1.1
- net GND: now also TP?.1
Changed lines of the file:
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@@
 (kicad_sch (version 20211123) (generator eeschema)
   (paper "A4")
+  (junction (at 75.692 86.106) (diameter 0) (color 0 0 0 0)
+  )
   (junction (at 42.926 181.102) (diameter 0) (color 0 0 0 0)
   )
@@
   )
   (junction (at 46.736 181.102) (diameter 0) (color 0 0 0 0)
+  )
+  (junction (at 84.328 83.566) (diameter 0) (color 0 0 0 0)
   )
   (no_connect (at 46.228 106.426))
   (no_connect (at 46.228 108.966))
+  (wire (pts (xy 30.988 116.586) (xy 52.324 116.586))
+    (stroke (width 0) (type default) (color 0 0 0 0))
+  )
   (wire (pts (xy 35.306 181.102) (xy 42.926 181.102))
     (stroke (width 0) (type default) (color 0 0 0 0))
@@
     (stroke (width 0) (type default) (color 0 0 0 0))
   )
+  (wire (pts (xy 52.324 116.586) (xy 52.324 113.792))
+    (stroke (width 0) (type default) (color 0 0 0 0))
+  )
   (wire (pts (xy 46.228 98.806) (xy 46.228 97.028))
     (stroke (width 0) (type default) (color 0 0 0 0))
@@
     (stroke (width 0) (type default) (color 0 0 0 0))
   )
+  (wire (pts (xy 75.692 73.152) (xy 75.692 86.106))
+    (stroke (width 0) (type default) (color 0 0 0 0))
+  )
   (wire (pts (xy 46.228 92.964) (xy 53.594 92.964))
     (stroke (width 0) (type default) (color 0 0 0 0))
@@
     (stroke (width 0) (type default) (color 0 0 0 0))
   )
-  (wire (pts (xy 46.228 86.106) (xy 76.2 86.106))
+  (wire (pts (xy 75.692 86.106) (xy 76.2 86.106))
+    (stroke (width 0) (type default) (color 0 0 0 0))
+  )
+  (wire (pts (xy 46.228 86.106) (xy 75.692 86.106))
     (stroke (width 0) (type default) (color 0 0 0 0))
   )
@@
   )
   (text "A Type-C host with 3A capability will have 10 k pull-up to 5 V,\na 1.5 A capability will be advertised with 22k pull-up, \nand the standard port capability (500 mA) will have 56 k pull-up."
-    (at 55.118 80.772 0)
+    (at 22.098 50.038 0)
     (effects (font (size 1.27 1.27)) (justify left bottom))
   )
@@
     (pin "2")
   )
+  (symbol (lib_id "Connector:TestPoint") (at 75.692 73.152 0) (unit 1)
+    (in_bom yes) (on_board yes) (fields_autoplaced)
+    (property "Reference" "TP1" (id 0) (at 77.47 68.5799 0)
+      (effects (font (size 1.27 1.27)) (justify left))
+    )
+    (property "Value" "TestPoint" (id 1) (at 77.47 71.1199 0)
+      (effects (font (size 1.27 1.27)) (justify left))
+    )
+    (property "Footprint" "TestPoint:TestPoint_Pad_D2.0mm" (id 2) (at 80.772 73.152 0)
+      (effects (font (size 1.27 1.27)) hide)
+    )
+    (property "Datasheet" "~" (id 3) (at 80.772 73.152 0)
+      (effects (font (size 1.27 1.27)) hide)
+    )
+    (pin "1")
+  )
+  (symbol (lib_id "Connector:TestPoint") (at 52.324 113.792 0) (unit 1)
+    (in_bom yes) (on_board yes) (fields_autoplaced)
+    (property "Reference" "TP?" (id 0) (at 54.356 109.2199 0)
+      (effects (font (size 1.27 1.27)) (justify left))
+    )
+    (property "Value" "TestPoint" (id 1) (at 54.356 111.7599 0)
+      (effects (font (size 1.27 1.27)) (justify left))
+    )
+    (property "Footprint" "TestPoint:TestPoint_Pad_D2.0mm" (id 2) (at 57.404 113.792 0)
+      (effects (font (size 1.27 1.27)) hide)
+    )
+    (property "Datasheet" "~" (id 3) (at 57.404 113.792 0)
+      (effects (font (size 1.27 1.27)) hide)
+    )
+    (pin "1")
+  )
   (symbol (lib_id "power:GND") (at 84.328 103.124 0) (unit 1)
     (in_bom yes) (on_board yes)
@@
     (pin "1")
     (pin "2")
+  )
+  (symbol (lib_id "Connector:TestPoint") (at 84.328 83.566 0) (unit 1)
+    (in_bom yes) (on_board yes) (fields_autoplaced)
+    (property "Reference" "TP2" (id 0) (at 86.36 78.9939 0)
+      (effects (font (size 1.27 1.27)) (justify left))
+    )
+    (property "Value" "TestPoint" (id 1) (at 86.36 81.5339 0)
+      (effects (font (size 1.27 1.27)) (justify left))
+    )
+    (property "Footprint" "TestPoint:TestPoint_Pad_D2.0mm" (id 2) (at 89.408 83.566 0)
+      (effects (font (size 1.27 1.27)) hide)
+    )
+    (property "Datasheet" "~" (id 3) (at 89.408 83.566 0)
+      (effects (font (size 1.27 1.27)) hide)
+    )
+    (pin "1")
   )
   (symbol (lib_id "Device:Polyfuse") (at 48.514 68.072 0) (unit 1)
@@
       (reference "SW1") (unit 1) (value "SW_Push") (footprint "Local:TS-1187A-B-A-B")
     )
+    (path "/4963feca-a4fe-4e8d-b8f3-d8047749fda5"
+      (reference "TP1") (unit 1) (value "TestPoint") (footprint "TestPoint:TestPoint_Pad_D2.0mm")
+    )
+    (path "/bfe0e104-4081-4d23-847f-8dd10eb0a278"
+      (reference "TP2") (unit 1) (value "TestPoint") (footprint "TestPoint:TestPoint_Pad_D2.0mm")
+    )
+    (path "/51395e73-8df1-47a4-93df-260d5f9ddad0"
+      (reference "TP?") (unit 1) (value "TestPoint") (footprint "TestPoint:TestPoint_Pad_D2.0mm")
+    )
     (path "/396ef3b4-140c-4bca-bc40-a1de8b38dc5a"

Commit message: feature creep
Parts:
- added J4, J?: USB_A, Local:UE27AE54100, symbol Connector:USB_A
- added U3: USB2514B_Bi, Package_DFN_QFN:QFN-36-1EP_6x6mm_P0.5mm_EP3.7x3.7mm, symbol Interface_USB:USB2514B_Bi
- TP1, TP2: footprint TestPoint:TestPoint_Pad_D2.0mm -> TestPoint:TestPoint_Pad_D1.0mm
- gave numbers to parts that had none: 1
Connections:
- net VBUS: no longer R13.1
- new net VIN: R13.1

Commit message: ready for JLCPCB
Parts:
- removed J4, J?: USB_A, Local:UE27AE54100, symbol Connector:USB_A
- removed U3: USB2514B_Bi, Package_DFN_QFN:QFN-36-1EP_6x6mm_P0.5mm_EP3.7x3.7mm, symbol Interface_USB:USB2514B_Bi
- F1: now left out of the parts list
- R13: footprint Resistor_SMD:R_0402_1005Metric -> Resistor_SMD:R_0603_1608Metric; LCSC (none) -> C13167
- renumbered TP2 to CC1, TP1 to CC2, TP3 to GND1
